Commit message: $ Wheels added and Chassis modified

File: description/gazebo_control.xacro (robot description, xacro)
@@ -4,6 +4,8 @@
 		<plugin name='diff_drive' filename='libgazebo_ros_diff_drive.so'>
 			<!-- Wheel Information -->
-			<left_joint>left_wheel_joint</left_joint>
-			<right_joint>right_wheel_joint</right_joint>
+			<left_joint>left_wheel_front_joint</left_joint>
+			<left_joint>left_wheel_back_joint</left_joint>
+			<right_joint>right_wheel_front_joint</right_joint>
+			<right_joint>right_wheel_back_joint</right_joint>
 			<wheel_separation>0.35</wheel_separation>
 			<wheel_diameter>0.1</wheel_diameter>

File: description/robot_core.xacro (robot description, xacro)
@@ -1,44 +1,45 @@
 <?xml version="1.0"?>
-<robot xmlns:xacro="http://www.ros.org/wiki/xacro" >
+<robot xmlns:xacro="http://www.ros.org/wiki/xacro">
 	<xacro:include filename="inertial_macros.xacro" />
 	<material name="white">
-    		<color rgba="1 1 1 1"/>
+		<color rgba="1 1 1 1"/>
 	</material>
 	<material name="orange">
-    		<color rgba="1 0.3 0.1 1"/>
+		<color rgba="1 0.3 0.1 1"/>
 	</material>
 	<material name="blue">
-    		<color rgba="0.2 0.2 1 1"/>
+		<color rgba="0.2 0.2 1 1"/>
 	</material>
 	<material name="black">
-    		<color rgba="0 0 0 1"/>
+		<color rgba="0 0 0 1"/>
 	</material>
 	<material name="red">
 		<color rgba="1 0 0 1"/>
 	</material>
-	<link name="base_link">
-	</link>
+	<!-- BASE LINK DECLARATION -->
+	<link name="base_link" />
+	<!-- CHASSIS MODELING -->
 	<joint name="chassis_joint" type="fixed">
-    		<parent link="base_link"/>
-    		<child link="chassis"/>
-    		<origin xyz="-0.1 0 0"/>
+		<parent link="base_link"/>
+		<child link="chassis"/>
+		<origin xyz="0 0 0"/>
 	</joint>
 	<link name="chassis">
-    		<visual>
-        		<origin xyz="0.15 0 0.075" rpy="0 0 0"/>
-        		<geometry>
-            			<box size="0.3 0.3 0.15"/>
-        		</geometry>
-        		<material name="white"/>
-    		</visual>
+		<visual>
+			<origin xyz="0 0 0" rpy="0 0 0"/>
+			<geometry>
+				<box size="0.5 0.3 0.15"/>
+			</geometry>
+			<material name="white"/>
+		</visual>
 		<collision>
-			<origin xyz="0.15 0 0.075" rpy="0 0 0"/>
+			<origin xyz="0 0 0" rpy="0 0 0"/>
 			<geometry>
-				<box size="0.3 0.3 0.15"/>
+				<box size="0.5 0.3 0.15"/>
 			</geometry>
 			<material name="white"/>
 		</collision>
-		<xacro:inertial_box mass="0.5" x="0.3" y="0.3" z="0.15">
-			<origin xyz="0.15 0 0.075" rpy="0 0 0"/>
+		<xacro:inertial_box mass="0.5" x="0.5" y="0.3" z="0.15">
+			<origin xyz="0 0 0" rpy="0 0 0"/>
 		</xacro:inertial_box>
 	</link>
@@ -46,21 +47,21 @@
 		<material>Gazebo/White</material>
 	</gazebo>
-	<!-- LEFT WHEEL -->
-	<joint name="left_wheel_joint" type="continuous">
-    		<parent link="base_link"/>
-    		<child link="left_wheel"/>
-    		<origin xyz="0 0.175 0" rpy="-${pi/2} 0 0"/>
-    		<axis xyz="0 0 1"/>
+	<!-- LEFT WHEELS -->
+	<joint name="left_wheel_front_joint" type="continuous">
+		<parent link="chassis"/>
+		<child link="left_wheel_front"/>
+		<origin xyz="0.2 0.175 -0.075" rpy="-${pi/2} 0 0"/>
+		<axis xyz="0 0 1"/>
 	</joint>
-	<link name="left_wheel">
-    		<visual>
-        		<geometry>
-            			<cylinder length="0.04" radius="0.05" />/>
-        		</geometry>
-        		<material name="blue"/>
-    		</visual>
+	<link name="left_wheel_front">
+		<visual>
+			<geometry>
+				<cylinder length="0.04" radius="0.05" />
+			</geometry>
+			<material name="blue"/>
+		</visual>
 		<collision>
 			<geometry>
-				<cylinder length="0.04" radius="0.05" />/>
+				<cylinder length="0.04" radius="0.05" />
 			</geometry>
 		</collision>
@@ -69,24 +70,49 @@
 		</xacro:inertial_cylinder>
 	</link>
-	<gazebo reference="left_wheel">
+	<gazebo reference="left_wheel_front">
 		<material>Gazebo/Blue</material>
 	</gazebo>
-	<!-- RIGHT WHEEL -->
-	<joint name="right_wheel_joint" type="continuous">
-    		<parent link="base_link"/>
-    		<child link="right_wheel"/>
-    		<origin xyz="0 -0.175 0" rpy="${pi/2} 0 0"/>
-    		<axis xyz="0 0 -1"/>
+	<joint name="left_wheel_back_joint" type="continuous">
+		<parent link="chassis"/>
+		<child link="left_wheel_back"/>
+		<origin xyz="-0.2 0.175 -0.075" rpy="-${pi/2} 0 0"/>
+		<axis xyz="0 0 1"/>
 	</joint>
-	<link name="right_wheel">
-    		<visual>
-        		<geometry>
-            			<cylinder length="0.04" radius="0.05" />/>
-        		</geometry>
-        		<material name="blue"/>
-    		</visual>
+	<link name="left_wheel_back">
+		<visual>
+			<geometry>
+				<cylinder length="0.04" radius="0.05" />
+			</geometry>
+			<material name="blue"/>
+		</visual>
 		<collision>
 			<geometry>
-				<cylinder length="0.04" radius="0.05" />/>
+				<cylinder length="0.04" radius="0.05" />
+			</geometry>
+		</collision>
+		<xacro:inertial_cylinder mass="0.1" length="0.05" radius="0.05">
+			<origin xyz="0 0 0" rpy="0 0 0"/>
+		</xacro:inertial_cylinder>
+	</link>
+	<gazebo reference="left_wheel_back">
+		<material>Gazebo/Blue</material>
+	</gazebo>
+	<!-- RIGHT WHEELS -->
+	<joint name = "right_wheel_front_joint" type = "continuous">
+		<parent link = "base_link"/>
+		<child link = "right_wheel_front"/>
+		<origin xyz = "0.2 -0.175 -0.075" rpy = "${pi/2} 0 0"/>
+		<axis xyz = "0 0 -1"/>
+	</joint>
+	<link name="right_wheel_front">
+		<visual>
+			<geometry>
+				<cylinder length="0.04" radius="0.05" />
+			</geometry>
+			<material name="blue"/>
+		</visual>
+		<collision>
+			<geometry>
+				<cylinder length="0.04" radius="0.05" />
 			</geometry>
 		</collision>
@@ -95,9 +121,34 @@
 		</xacro:inertial_sphere>
 	</link>
-	<gazebo reference="right_wheel">
+	<gazebo reference="right_wheel_front">
+		<material>Gazebo/Blue</material>
+	</gazebo>
+	<joint name="right_wheel_back_joint" type="continuous">
+		<parent link="base_link"/>
+		<child link="right_wheel_back"/>
+		<origin xyz="-0.2 -0.175 -0.075" rpy="${pi/2} 0 0"/>
+		<axis xyz="0 0 -1"/>
+	</joint>
+	<link name="right_wheel_back">
+		<visual>
+			<geometry>
+				<cylinder length = "0.04" radius = "0.05" />
+			</geometry>
+			<material name="blue"/>
+		</visual>
+		<collision>
+			<geometry>
+				<cylinder length = "0.04" radius = "0.05" />
+			</geometry>
+		</collision>
+		<xacro:inertial_sphere mass = "0.1" radius = "0.05">
+			<origin xyz="0 0 0" rpy="0 0 0"/>
+		</xacro:inertial_sphere>
+	</link>
+	<gazebo reference="right_wheel_back">
 		<material>Gazebo/Blue</material>
 	</gazebo>
 	<!-- CASTER WHEEL -->
-	<joint name="caster_wheel_joint" type="fixed">
+	<!--<joint name="caster_wheel_joint" type="fixed">
 		<parent link="chassis"/>
 		<child link="caster_wheel"/>
@@ -121,4 +172,4 @@
 		<mu1 value="0.001"/>
 		<mu2 value="0.001"/>
-	</gazebo>
+	</gazebo>-->
 </robot>

File: description/ros2_control.xacro (robot description, xacro)
@@ -5,5 +5,5 @@
 			<plugin>gazebo_ros2_control/GazeboSystem</plugin>
 		</hardware>
-		<joint name="left_wheel_joint">
+		<joint name="left_wheel_front_joint">
 			<command_interface name="velocity">
 				<param name="min">-10</param>
@@ -13,5 +13,21 @@
 			<state_interface name="velocity" />
 		</joint>
-		<joint name="right_wheel_joint">
+		<joint name="left_wheel_back_joint">
+			<command_interface name="velocity">
+				<param name="min">-10</param>
+				<param name="max">10</param>
+			</command_interface>
+			<state_interface name="position" />
+			<state_interface name="velocity" />
+		</joint>
+		<joint name="right_wheel_front_joint">
+			<command_interface name="velocity">
+				<param name="min">-10</param>
+				<param name="max">10</param>
+			</command_interface>
+			<state_interface name="velocity" />
+			<state_interface name="position" />
+		</joint>
+		<joint name="right_wheel_back_joint">
 			<command_interface name="velocity">
 				<param name="min">-10</param>

Commit message: Implemented a somehow working 4WD

File: description/gazebo_control.xacro (robot description, xacro)
@@ -2,10 +2,14 @@
 <robot xmlns:xacro="http://www.ros.org/wiki/xacro">
 	<gazebo>
-		<plugin name='diff_drive' filename='libgazebo_ros_diff_drive.so'>
+		<plugin name = 'diff_drive' filename = 'libgazebo_ros_diff_drive.so'>
 			<!-- Wheel Information -->
-			<left_joint>left_wheel_front_joint</left_joint>
-			<left_joint>left_wheel_back_joint</left_joint>
-			<right_joint>right_wheel_front_joint</right_joint>
-			<right_joint>right_wheel_back_joint</right_joint>
+			<left_joint>
+				left_wheel_front_joint
+				left_wheel_back_joint
+			</left_joint>
+			<right_joint>
+				right_wheel_front_joint
+				right_wheel_back_joint
+			</right_joint>
 			<wheel_separation>0.35</wheel_separation>
 			<wheel_diameter>0.1</wheel_diameter>

File: description/robot_core.xacro (robot description, xacro)
@@ -2,11 +2,12 @@
 <robot xmlns:xacro="http://www.ros.org/wiki/xacro">
 	<xacro:include filename="inertial_macros.xacro" />
-	<material name="white"> <color rgba="1 1 1 1"/> </material>
-	<material name="orange"> <color rgba="1 0.3 0.1 1"/> </material>
-	<material name="blue"> <color rgba="0.2 0.2 1 1"/> </material>
-	<material name="black"> <color rgba="0 0 0 1"/> </material>
-	<material name="red"> <color rgba="1 0 0 1"/> </material>
+	<material name="white"> <color rgba = "1 1 1 1"/> </material>
+	<material name="orange"> <color rgba = "1 0.3 0.1 1"/> </material>
+	<material name="blue"> <color rgba = "0.2 0.2 1 1"/> </material>
+	<material name="black"> <color rgba = "0 0 0 1"/> </material>
+	<material name="red"> <color rgba = "1 0 0 1"/> </material>
 	<!-- BASE LINK DECLARATION -->
-	<link name="base_link" />
+	<link name="base_link">
+	</link>
 	<!-- CHASSIS MODELING -->
 	<joint name="chassis_joint" type="fixed">
@@ -39,5 +40,5 @@
 	<!-- LEFT WHEELS -->
 	<joint name="left_wheel_front_joint" type="continuous">
-		<parent link="base_link"/>
+		<parent link="chassis"/>
 		<child link="left_wheel_front"/>
 		<origin xyz="0.2 0.175 -0.075" rpy="-${pi/2} 0 0"/>
@@ -64,5 +65,5 @@
 	</gazebo>
 	<joint name="left_wheel_back_joint" type="continuous">
-		<parent link="base_link"/>
+		<parent link="chassis"/>
 		<child link="left_wheel_back"/>
 		<origin xyz="-0.2 0.175 -0.075" rpy="-${pi/2} 0 0"/>
@@ -90,5 +91,5 @@
 	<!-- RIGHT WHEELS -->
 	<joint name = "right_wheel_front_joint" type = "continuous">
-		<parent link = "base_link"/>
+		<parent link = "chassis"/>
 		<child link = "right_wheel_front"/>
 		<origin xyz = "0.2 -0.175 -0.075" rpy = "${pi/2} 0 0"/>
@@ -115,5 +116,5 @@
 	</gazebo>
 	<joint name="right_wheel_back_joint" type="continuous">
-		<parent link="base_link"/>
+		<parent link="chassis"/>
 		<child link="right_wheel_back"/>
 		<origin xyz="-0.2 -0.175 -0.075" rpy="${pi/2} 0 0"/>
