Commit message: Gazeo Control

File: description/robot.urdf.xacro (robot description, xacro)
@@ -1,5 +1,5 @@
 <?xml version="1.0"?>
 <robot xmlns:xacro="http://www.ros.org/wiki/xacro"  name="robot">
-	<xacro:include filename="robot_core.xacro" />
-	<xacro:include filename="inertial_macros.xacro" /> <!-- NOT WORKING-->
+    <xacro:include filename="robot_core.xacro" />
+	<xacro:include filename="gazebo_control.xacro" />
 </robot>

File: description/robot_core.xacro (robot description, xacro)
@@ -40,4 +40,7 @@
 		</xacro:inertial_box>
 	</link>
+	<gazebo reference="chassis">
+		<material>Gazebo/White</material>
+	</gazebo>
 	<!-- LEFT WHEEL -->
 	<joint name="left_wheel_joint" type="continuous">
@@ -63,4 +66,7 @@
 		</xacro:inertial_cylinder>
 	</link>
+	<gazebo reference="left_wheel">
+		<material>Gazebo/Blue</material>
+	</gazebo>
 	<!-- RIGHT WHEEL -->
 	<joint name="right_wheel_joint" type="continuous">
@@ -86,4 +92,7 @@
 		</xacro:inertial_sphere>
 	</link>
+	<gazebo reference="right_wheel">
+		<material>Gazebo/Blue</material>
+	</gazebo>
 	<!-- CASTER WHEEL -->
 	<joint name="caster_wheel_joint" type="fixed">
@@ -105,3 +114,8 @@
 		</collision>
 	</link>
+	<gazebo reference="caster_wheel">
+		<material>Gazebo/Black</material>
+		<mu1 value="0.001"/>
+		<mu2 value="0.001"/>
+	</gazebo>
 </robot>

Commit message: LiDAR Sim

File: description/robot.urdf.xacro (robot description, xacro)
@@ -3,3 +3,4 @@
     <xacro:include filename="robot_core.xacro" />
 	<xacro:include filename="gazebo_control.xacro" />
+	<xacro:include filename="lidar.xacro" />
 </robot>

File: description/robot_core.xacro (robot description, xacro)
@@ -13,4 +13,7 @@
 	<material name="black">
     		<color rgba="0 0 0 1"/>
+	</material>
+	<material name="red">
+		<color rgba="1 0 0 1"/>
 	</material>
 	<link name="base_link">

Commit message: test

File: description/robot.urdf.xacro (robot description, xacro)
@@ -2,7 +2,7 @@
 <robot xmlns:xacro="http://www.ros.org/wiki/xacro"  name="robot">
     <xacro:include filename="robot_core.xacro" />
+	<xacro:include filename="ros2_control.xacro" />
 	<!-- <xacro:include filename="gazebo_control.xacro" /> -->
 	<!-- <xacro:include filename="lidar.xacro" /> -->
-	<xacro:include filename="camera.xacro" />
-	<xacro:include filename="ros2_control.xacro" />
+	<!-- <xacro:include filename="camera.xacro" /> -->
 </robot>

File: description/robot_core.xacro (robot description, xacro)
@@ -8,5 +8,6 @@
 	<material name="red"> <color rgba = "1 0 0 1"/> </material>
 	<!-- BASE LINK DECLARATION -->
-	<link name="base_link">
+	<link name="base_link" >
+		<origin xyz = "0.0 0.175 -0.075"/>
 	</link>
 	<!-- CHASSIS MODELING -->
@@ -40,5 +41,5 @@
 	<!-- LEFT WHEELS -->
 	<joint name="left_wheel_front_joint" type="continuous">
-		<parent link="chassis"/>
+		<parent link="base_link"/>
 		<child link="left_wheel_front"/>
 		<origin xyz="0.2 0.175 -0.075" rpy="-${pi/2} 0 0"/>
@@ -65,5 +66,5 @@
 	</gazebo>
 	<joint name="left_wheel_back_joint" type="continuous">
-		<parent link="chassis"/>
+		<parent link="base_link"/>
 		<child link="left_wheel_back"/>
 		<origin xyz="-0.2 0.175 -0.075" rpy="-${pi/2} 0 0"/>
@@ -91,8 +92,8 @@
 	<!-- RIGHT WHEELS -->
 	<joint name = "right_wheel_front_joint" type = "continuous">
-		<parent link = "chassis"/>
+		<parent link = "base_link"/>
 		<child link = "right_wheel_front"/>
 		<origin xyz = "0.2 -0.175 -0.075" rpy = "${pi/2} 0 0"/>
-		<axis xyz = "0 0 -1"/>
+		<axis xyz = "0 0 1"/>
 	</joint>
 	<link name="right_wheel_front">
@@ -116,8 +117,8 @@
 	</gazebo>
 	<joint name="right_wheel_back_joint" type="continuous">
-		<parent link="chassis"/>
+		<parent link="base_link"/>
 		<child link="right_wheel_back"/>
 		<origin xyz="-0.2 -0.175 -0.075" rpy="${pi/2} 0 0"/>
-		<axis xyz="0 0 -1"/>
+		<axis xyz="0 0 1"/>
 	</joint>
 	<link name="right_wheel_back">
@@ -140,27 +141,3 @@
 		<material>Gazebo/Blue</material>
 	</gazebo>
-	<!-- CASTER WHEEL -->
-	<!--<joint name="caster_wheel_joint" type="fixed">
-		<parent link="chassis"/>
-		<child link="caster_wheel"/>
-		<origin xyz="0.24 0 0" rpy="0 0 0"/>
-	</joint>
-	<link name="caster_wheel">
-		<visual>
-			<geometry>
-				<sphere radius="0.05" />
-			</geometry>
-			<material name="black"/>
-		</visual>
-		<collision>
-			<geometry>
-				<sphere radius="0.05" />
-			</geometry>
-		</collision>
-	</link>
-	<gazebo reference="caster_wheel">
-		<material>Gazebo/Black</material>
-		<mu1 value="0.001"/>
-		<mu2 value="0.001"/>
-	</gazebo>-->
 </robot>
