Commit message: updated controller yaml

File: description/robot_core.xacro (robot description, xacro)
@@ -2,19 +2,9 @@
 <robot xmlns:xacro="http://www.ros.org/wiki/xacro">
 	<xacro:include filename="inertial_macros.xacro" />
-	<material name="white">
-		<color rgba="1 1 1 1"/>
-	</material>
-	<material name="orange">
-		<color rgba="1 0.3 0.1 1"/>
-	</material>
-	<material name="blue">
-		<color rgba="0.2 0.2 1 1"/>
-	</material>
-	<material name="black">
-		<color rgba="0 0 0 1"/>
-	</material>
-	<material name="red">
-		<color rgba="1 0 0 1"/>
-	</material>
+	<material name="white"> <color rgba="1 1 1 1"/> </material>
+	<material name="orange"> <color rgba="1 0.3 0.1 1"/> </material>
+	<material name="blue"> <color rgba="0.2 0.2 1 1"/> </material>
+	<material name="black"> <color rgba="0 0 0 1"/> </material>
+	<material name="red"> <color rgba="1 0 0 1"/> </material>
 	<!-- BASE LINK DECLARATION -->
 	<link name="base_link" />

File: description/ros2_control.xacro (robot description, xacro)
@@ -1,43 +1,43 @@
 ﻿<?xml version="1.0"?>
 <robot xmlns:xacro="http://www.ros.org/wiki/xacro">
-	<ros2_control name="GazeboSystem" type="system">
+	<ros2_control name = "GazeboSystem" type = "system">
 		<hardware>
 			<plugin>gazebo_ros2_control/GazeboSystem</plugin>
 		</hardware>
-		<joint name="left_wheel_front_joint">
-			<command_interface name="velocity">
-				<param name="min">-10</param>
-				<param name="max">10</param>
+		<joint name = "left_wheel_front_joint">
+			<command_interface name = "velocity">
+				<param name = "min"> -10 </param>
+				<param name = "max"> 10 </param>
 			</command_interface>
-			<state_interface name="position" />
-			<state_interface name="velocity" />
+			<state_interface name = "position" />
+			<state_interface name = "velocity" />
 		</joint>
-		<joint name="left_wheel_back_joint">
-			<command_interface name="velocity">
-				<param name="min">-10</param>
-				<param name="max">10</param>
+		<joint name = "left_wheel_back_joint">
+			<command_interface name = "velocity">
+				<param name = "min"> -10 </param>
+				<param name = "max"> 10 </param>
 			</command_interface>
-			<state_interface name="position" />
-			<state_interface name="velocity" />
+			<state_interface name = "position" />
+			<state_interface name = "velocity" />
 		</joint>
-		<joint name="right_wheel_front_joint">
-			<command_interface name="velocity">
-				<param name="min">-10</param>
-				<param name="max">10</param>
+		<joint name = "right_wheel_front_joint">
+			<command_interface name = "velocity">
+				<param name = "min"> -10 </param>
+				<param name = "max"> 10 </param>
 			</command_interface>
-			<state_interface name="velocity" />
-			<state_interface name="position" />
+			<state_interface name = "velocity" />
+			<state_interface name = "position" />
 		</joint>
-		<joint name="right_wheel_back_joint">
-			<command_interface name="velocity">
-				<param name="min">-10</param>
-				<param name="max">10</param>
+		<joint name = "right_wheel_back_joint">
+			<command_interface name = "velocity">
+				<param name = "min"> -10 </param>
+				<param name = "max"> 10 </param>
 			</command_interface>
-			<state_interface name="velocity" />
-			<state_interface name="position" />
+			<state_interface name = "velocity" />
+			<state_interface name = "position" />
 		</joint>
 	</ros2_control>
 	<gazebo>
-		<plugin filename="libgazebo_ros2_control.so" name="gazebo_ros2_control">
+		<plugin filename = "libgazebo_ros2_control.so" name = "gazebo_ros2_control">
 			<parameters>
 				$(find rosbot)/config/my_controllers.yaml

Commit message: logic fix

File: description/robot_core.xacro (robot description, xacro)
@@ -39,5 +39,5 @@
 	<!-- LEFT WHEELS -->
 	<joint name="left_wheel_front_joint" type="continuous">
-		<parent link="chassis"/>
+		<parent link="base_link"/>
 		<child link="left_wheel_front"/>
 		<origin xyz="0.2 0.175 -0.075" rpy="-${pi/2} 0 0"/>
@@ -64,5 +64,5 @@
 	</gazebo>
 	<joint name="left_wheel_back_joint" type="continuous">
-		<parent link="chassis"/>
+		<parent link="base_link"/>
 		<child link="left_wheel_back"/>
 		<origin xyz="-0.2 0.175 -0.075" rpy="-${pi/2} 0 0"/>

Commit message: Changed joints and some fixes

File: description/robot_core.xacro (robot description, xacro)
@@ -1,37 +1,35 @@
 <?xml version="1.0"?>
-<robot xmlns:xacro="http://www.ros.org/wiki/xacro">
-	<xacro:include filename="inertial_macros.xacro" />
-	<material name="white"> <color rgba = "1 1 1 1"/> </material>
-	<material name="orange"> <color rgba = "1 0.3 0.1 1"/> </material>
-	<material name="blue"> <color rgba = "0.2 0.2 1 1"/> </material>
-	<material name="black"> <color rgba = "0 0 0 1"/> </material>
-	<material name="red"> <color rgba = "1 0 0 1"/> </material>
+<robot xmlns:xacro = "http://www.ros.org/wiki/xacro">
+	<xacro:include filename = "inertial_macros.xacro" />
+	<material name = "white"> <color rgba = "1 1 1 1"/> </material>
+	<material name = "orange"> <color rgba = "1 0.3 0.1 1"/> </material>
+	<material name = "blue"> <color rgba = "0.2 0.2 1 1"/> </material>
+	<material name = "black"> <color rgba = "0 0 0 1"/> </material>
+	<material name = "red"> <color rgba = "1 0 0 1"/> </material>
 	<!-- BASE LINK DECLARATION -->
-	<link name="base_link" >
-		<origin xyz = "0.0 0.175 -0.075"/>
-	</link>
+	<link name = "base_link" />
 	<!-- CHASSIS MODELING -->
-	<joint name="chassis_joint" type="fixed">
-		<parent link="base_link"/>
-		<child link="chassis"/>
-		<origin xyz="0 0 0"/>
+	<joint name = "chassis_joint" type="fixed">
+		<parent link = "base_link"/>
+		<child link = "chassis"/>
+		<origin xyz = "-0.1 0 0"/>
 	</joint>
-	<link name="chassis">
+	<link name = "chassis">
 		<visual>
-			<origin xyz="0 0 0" rpy="0 0 0"/>
+			<origin xyz = "0.25 0 0.075" rpy = "0 0 0"/>
 			<geometry>
-				<box size="0.5 0.3 0.15"/>
+				<box size = "0.5 0.3 0.15"/>
 			</geometry>
-			<material name="white"/>
+			<material name = "white"/>
 		</visual>
 		<collision>
-			<origin xyz="0 0 0" rpy="0 0 0"/>
+			<origin xyz = "0.25 0 0.075" rpy="0 0 0"/>
 			<geometry>
-				<box size="0.5 0.3 0.15"/>
+				<box size = "0.5 0.3 0.15"/>
 			</geometry>
-			<material name="white"/>
+			<material name = "white"/>
 		</collision>
-		<xacro:inertial_box mass="0.5" x="0.5" y="0.3" z="0.15">
-			<origin xyz="0 0 0" rpy="0 0 0"/>
+		<xacro:inertial_box mass = "0.5" x = "0.5" y = "0.3" z = "0.15">
+			<origin xyz = "0.25 0 0.075" rpy = "0 0 0"/>
 		</xacro:inertial_box>
 	</link>
@@ -40,24 +38,24 @@
 	</gazebo>
 	<!-- LEFT WHEELS -->
-	<joint name="left_wheel_front_joint" type="continuous">
-		<parent link="base_link"/>
-		<child link="left_wheel_front"/>
-		<origin xyz="0.2 0.175 -0.075" rpy="-${pi/2} 0 0"/>
-		<axis xyz="0 0 1"/>
+	<joint name = "left_wheel_front_joint" type = "continuous">
+		<parent link = "base_link"/>
+		<child link = "left_wheel_front"/>
+		<origin xyz = "0.3 0.175 0" rpy = "-${pi/2} 0 0"/>
+		<axis xyz = "0 0 1"/>
 	</joint>
-	<link name="left_wheel_front">
+	<link name = "left_wheel_front">
 		<visual>
 			<geometry>
-				<cylinder length="0.04" radius="0.05" />
+				<cylinder length = "0.04" radius = "0.05" />
 			</geometry>
-			<material name="blue"/>
+			<material name = "blue"/>
 		</visual>
 		<collision>
 			<geometry>
-				<cylinder length="0.04" radius="0.05" />
+				<cylinder length = "0.04" radius = "0.05" />
 			</geometry>
 		</collision>
-		<xacro:inertial_cylinder mass="0.1" length="0.05" radius="0.05">
-			<origin xyz="0 0 0" rpy="0 0 0"/>
+		<xacro:inertial_cylinder mass = "0.1" length = "0.05" radius = "0.05">
+			<origin xyz = "0 0 0" rpy = "0 0 0"/>
 		</xacro:inertial_cylinder>
 	</link>
@@ -68,5 +66,5 @@
 		<parent link="base_link"/>
 		<child link="left_wheel_back"/>
-		<origin xyz="-0.2 0.175 -0.075" rpy="-${pi/2} 0 0"/>
+		<origin xyz="0 0.175 0" rpy="-${pi/2} 0 0"/>
 		<axis xyz="0 0 1"/>
 	</joint>
@@ -80,9 +78,9 @@
 		<collision>
 			<geometry>
-				<cylinder length="0.04" radius="0.05" />
+				<cylinder length = "0.04" radius = "0.05" />
 			</geometry>
 		</collision>
-		<xacro:inertial_cylinder mass="0.1" length="0.05" radius="0.05">
-			<origin xyz="0 0 0" rpy="0 0 0"/>
+		<xacro:inertial_cylinder mass = "0.1" length = "0.05" radius = "0.05">
+			<origin xyz = "0 0 0" rpy = "0 0 0"/>
 		</xacro:inertial_cylinder>
 	</link>
@@ -94,6 +92,6 @@
 		<parent link = "base_link"/>
 		<child link = "right_wheel_front"/>
-		<origin xyz = "0.2 -0.175 -0.075" rpy = "${pi/2} 0 0"/>
-		<axis xyz = "0 0 1"/>
+		<origin xyz = "0.3 -0.175 0" rpy = "${pi/2} 0 0"/>
+		<axis xyz = "0 0 -1"/>
 	</joint>
 	<link name="right_wheel_front">
@@ -109,7 +107,7 @@
 			</geometry>
 		</collision>
-		<xacro:inertial_sphere mass="0.1" radius="0.05">
-			<origin xyz="0 0 0" rpy="0 0 0"/>
-		</xacro:inertial_sphere>
+		<xacro:inertial_cylinder mass = "0.1" length = "0.05" radius = "0.05">
+			<origin xyz = "0 0 0" rpy = "0 0 0"/>
+		</xacro:inertial_cylinder>
 	</link>
 	<gazebo reference="right_wheel_front">
@@ -119,6 +117,6 @@
 		<parent link="base_link"/>
 		<child link="right_wheel_back"/>
-		<origin xyz="-0.2 -0.175 -0.075" rpy="${pi/2} 0 0"/>
-		<axis xyz="0 0 1"/>
+		<origin xyz="0 -0.175 0" rpy="${pi/2} 0 0"/>
+		<axis xyz="0 0 -1"/>
 	</joint>
 	<link name="right_wheel_back">
@@ -134,7 +132,7 @@
 			</geometry>
 		</collision>
-		<xacro:inertial_sphere mass = "0.1" radius = "0.05">
-			<origin xyz="0 0 0" rpy="0 0 0"/>
-		</xacro:inertial_sphere>
+		<xacro:inertial_cylinder mass = "0.1" length = "0.05" radius = "0.05">
+			<origin xyz = "0 0 0" rpy = "0 0 0"/>
+		</xacro:inertial_cylinder>
 	</link>
 	<gazebo reference="right_wheel_back">
