Commit message: Added ROS control and some code corrections

File: description/camera.xacro (robot description, xacro)
@@ -9,5 +9,5 @@
 		<visual>
 			<geometry>
-				<box radius="0.010 0.03 0.03" length="0.04"/>
+				<box size="0.010 0.03 0.03"/>
 			</geometry>
 			<material name="red"/>

File: description/robot.urdf.xacro (robot description, xacro)
@@ -2,6 +2,7 @@
 <robot xmlns:xacro="http://www.ros.org/wiki/xacro"  name="robot">
     <xacro:include filename="robot_core.xacro" />
-	<xacro:include filename="gazebo_control.xacro" />
+	<!-- <xacro:include filename="gazebo_control.xacro" /> -->
 	<!-- <xacro:include filename="lidar.xacro" /> -->
 	<xacro:include filename="camera.xacro" />
+	<xacro:include filename="ros2_control.xacro" />
 </robot>

Commit message: Body modifications

File: description/camera.xacro (robot description, xacro)
@@ -4,5 +4,5 @@
 		<parent link="chassis"/>
 		<child link="camera_link"/>
-		<origin xyz="0.305 0 0.08" rpy="0 0 0"/>
+		<origin xyz="0.1 0 0.105" rpy="0 0 0"/>
 	</joint>
 	<link name="camera_link">
@@ -35,9 +35,9 @@
 			<update_rate>10</update_rate>
 			<camera>
-				<horizontal_fov>1.089</horizontal_fov>
+				<horizontal_fov>1.0472</horizontal_fov>
 				<image>
 					<format>R8G8B8</format>
 					<width>640</width>
-					<height>480</height>
+					<height>280</height>
 				</image>
 				<clip>

File: description/gazebo_control.xacro (robot description, xacro)
@@ -3,5 +3,5 @@
 	<gazebo>
 		<plugin name = 'diff_drive' filename = 'libgazebo_ros_diff_drive.so'>
-			<!-- Wheel Information -->
+			<num_wheel_pairs>2</num_wheel_pairs>
 			<left_joint>
 				left_wheel_front_joint
@@ -13,9 +13,7 @@
 			</right_joint>
 			<wheel_separation>0.35</wheel_separation>
-			<wheel_diameter>0.1</wheel_diameter>
-			<!-- Limits -->
+			<wheel_diameter>0.6</wheel_diameter>
 			<max_wheel_torque>200</max_wheel_torque>
-			<max_wheel_acceleration>10.0</max_wheel_acceleration>
-			<!-- Output -->
+			<max_wheel_acceleration>100.0</max_wheel_acceleration>
 			<odometry_frame>odom</odometry_frame>
 			<robot_base_frame>base_link</robot_base_frame>
@@ -25,3 +23,19 @@
 		</plugin>
 	</gazebo>
+	<!-- <gazebo>
+		<plugin name = "skid_steer_drive_controller" filename = "libgazebo_ros_skid_steer_drive.so">
+			<updateRate>30.0</updateRate>
+			<robotNamespace>/</robotNamespace>
+			<leftFrontJoint>front_left_wheel_joint</leftFrontJoint>
+			<rightFrontJoint>front_right_wheel_joint</rightFrontJoint>
+			<leftRearJoint>back_left_wheel_joint</leftRearJoint>
+			<rightRearJoint>back_right_wheel_joint</rightRearJoint>
+			<wheelSeparation>0.35</wheelSeparation>
+			<wheelDiameter>0.6</wheelDiameter>
+			<robotBaseFrame>base_link</robotBaseFrame>
+			<torque>200</torque>
+			<topicName>cmd_vel</topicName>
+			<broadcastTF>false</broadcastTF>
+		</plugin>
+	</gazebo> -->
 </robot>

File: description/robot.urdf.xacro (robot description, xacro)
@@ -1,8 +1,8 @@
-<?xml version="1.0"?>
-<robot xmlns:xacro="http://www.ros.org/wiki/xacro"  name="robot">
-    <xacro:include filename="robot_core.xacro" />
-	<xacro:include filename="ros2_control.xacro" />
-	<!-- <xacro:include filename="gazebo_control.xacro" /> -->
-	<!-- <xacro:include filename="lidar.xacro" /> -->
-	<!-- <xacro:include filename="camera.xacro" /> -->
+<?xml version = "1.0"?>
+<robot xmlns:xacro = "http://www.ros.org/wiki/xacro"  name = "robot">
+    <xacro:include filename = "robot_core.xacro" />
+	<xacro:include filename = "ros2_control.xacro" />
+	<!-- <xacro:include filename = "gazebo_control.xacro" /> -->
+	<!-- <xacro:include filename = "lidar.xacro" /> -->
+	<xacro:include filename = "camera.xacro" />
 </robot>

File: description/robot_core.xacro (robot description, xacro)
@@ -17,19 +17,19 @@
 	<link name = "chassis">
 		<visual>
-			<origin xyz = "0.25 0 0.075" rpy = "0 0 0"/>
+			<origin xyz = "0.115 0 0.045" rpy = "0 0 0"/>
 			<geometry>
-				<box size = "0.5 0.3 0.15"/>
+				<box size = "0.23 0.11 0.09"/>
 			</geometry>
 			<material name = "white"/>
 		</visual>
 		<collision>
-			<origin xyz = "0.25 0 0.075" rpy="0 0 0"/>
+			<origin xyz = "0.115 0 0.045" rpy="0 0 0"/>
 			<geometry>
-				<box size = "0.5 0.3 0.15"/>
+				<box size = "0.23 0.11 0.09"/>
 			</geometry>
 			<material name = "white"/>
 		</collision>
-		<xacro:inertial_box mass = "0.5" x = "0.5" y = "0.3" z = "0.15">
-			<origin xyz = "0.25 0 0.075" rpy = "0 0 0"/>
+		<xacro:inertial_box mass = "0.75" x = "0.23" y = "0.11" z = "0.09">
+			<origin xyz = "0.115 0 0.045" rpy = "0 0 0"/>
 		</xacro:inertial_box>
 	</link>
@@ -41,5 +41,5 @@
 		<parent link = "base_link"/>
 		<child link = "left_wheel_front"/>
-		<origin xyz = "0.3 0.175 0" rpy = "-${pi/2} 0 0"/>
+		<origin xyz = "0.095 0.0625 0" rpy = "-${pi/2} 0 0"/>
 		<axis xyz = "0 0 1"/>
 	</joint>
@@ -47,5 +47,5 @@
 		<visual>
 			<geometry>
-				<cylinder length = "0.04" radius = "0.05" />
+				<cylinder length = "0.015" radius = "0.03" />
 			</geometry>
 			<material name = "blue"/>
@@ -53,8 +53,8 @@
 		<collision>
 			<geometry>
-				<cylinder length = "0.04" radius = "0.05" />
+				<cylinder length = "0.015" radius = "0.03" />
 			</geometry>
 		</collision>
-		<xacro:inertial_cylinder mass = "0.1" length = "0.05" radius = "0.05">
+		<xacro:inertial_cylinder mass = "0.1" length = "0.015" radius = "0.03">
 			<origin xyz = "0 0 0" rpy = "0 0 0"/>
 		</xacro:inertial_cylinder>
@@ -66,5 +66,5 @@
 		<parent link="base_link"/>
 		<child link="left_wheel_back"/>
-		<origin xyz="0 0.175 0" rpy="-${pi/2} 0 0"/>
+		<origin xyz="-0.065 0.0625 0" rpy="-${pi/2} 0 0"/>
 		<axis xyz="0 0 1"/>
 	</joint>
@@ -72,5 +72,5 @@
 		<visual>
 			<geometry>
-				<cylinder length="0.04" radius="0.05" />
+				<cylinder length = "0.015" radius = "0.03" />
 			</geometry>
 			<material name="blue"/>
@@ -78,8 +78,8 @@
 		<collision>
 			<geometry>
-				<cylinder length = "0.04" radius = "0.05" />
+				<cylinder length = "0.015" radius = "0.03" />
 			</geometry>
 		</collision>
-		<xacro:inertial_cylinder mass = "0.1" length = "0.05" radius = "0.05">
+		<xacro:inertial_cylinder mass = "0.1" length = "0.015" radius = "0.03">
 			<origin xyz = "0 0 0" rpy = "0 0 0"/>
 		</xacro:inertial_cylinder>
@@ -92,5 +92,5 @@
 		<parent link = "base_link"/>
 		<child link = "right_wheel_front"/>
-		<origin xyz = "0.3 -0.175 0" rpy = "${pi/2} 0 0"/>
+		<origin xyz = "0.095 -0.0625 0" rpy = "${pi/2} 0 0"/>
 		<axis xyz = "0 0 -1"/>
 	</joint>
@@ -98,5 +98,5 @@
 		<visual>
 			<geometry>
-				<cylinder length="0.04" radius="0.05" />
+				<cylinder length = "0.015" radius="0.03" />
 			</geometry>
 			<material name="blue"/>
@@ -104,8 +104,8 @@
 		<collision>
 			<geometry>
-				<cylinder length="0.04" radius="0.05" />
+				<cylinder length = "0.015" radius="0.03" />
 			</geometry>
 		</collision>
-		<xacro:inertial_cylinder mass = "0.1" length = "0.05" radius = "0.05">
+		<xacro:inertial_cylinder mass = "0.1" length = "0.015" radius = "0.03">
 			<origin xyz = "0 0 0" rpy = "0 0 0"/>
 		</xacro:inertial_cylinder>
@@ -117,5 +117,5 @@
 		<parent link="base_link"/>
 		<child link="right_wheel_back"/>
-		<origin xyz="0 -0.175 0" rpy="${pi/2} 0 0"/>
+		<origin xyz="-0.065 -0.0625 0" rpy="${pi/2} 0 0"/>
 		<axis xyz="0 0 -1"/>
 	</joint>
@@ -123,5 +123,5 @@
 		<visual>
 			<geometry>
-				<cylinder length = "0.04" radius = "0.05" />
+				<cylinder length = "0.015" radius = "0.03" />
 			</geometry>
 			<material name="blue"/>
@@ -129,8 +129,8 @@
 		<collision>
 			<geometry>
-				<cylinder length = "0.04" radius = "0.05" />
+				<cylinder length = "0.015" radius = "0.03" />
 			</geometry>
 		</collision>
-		<xacro:inertial_cylinder mass = "0.1" length = "0.05" radius = "0.05">
+		<xacro:inertial_cylinder mass = "0.1" length = "0.015" radius = "0.03">
 			<origin xyz = "0 0 0" rpy = "0 0 0"/>
 		</xacro:inertial_cylinder>

File: description/ros2_control.xacro (robot description, xacro)
@@ -1,4 +1,4 @@
-﻿<?xml version="1.0"?>
-<robot xmlns:xacro="http://www.ros.org/wiki/xacro">
+﻿<?xml version = "1.0"?>
+<robot xmlns:xacro = "http://www.ros.org/wiki/xacro">
 	<ros2_control name = "GazeboSystem" type = "system">
 		<hardware>
